File: datasheets/transmitter/transmitter.kicad_pcb (KiCad board)
At the start: 2 copper layers, 8 parts, among them IC1 ATTINY85-P, Q1 Q_NPN_EBC

Commit message: Revert "Kicad PCB layout"
This reverts commit 9afb40ae9a6d2ea0d6b4d8b9758429dc2c52fee4.
Parts:
- removed ? (x2): , Wire_Pads:SolderWirePad_single_0-8mmDrill
- added REF**: Pin_Header_Straight_1x02, Pin_Headers:Pin_Header_Straight_1x02, F.Cu at (111.8, 109.2)
- added REF**: SolderWirePad_2x_0-8mmDrill, Wire_Pads:SolderWirePad_2x_0-8mmDrill, F.Cu at (128.3, 116.2)
- CON1: renamed from ?; value (none) -> AVR-ISP-6
- moved R2 8.52 mm to (107.3, 117.5), turned to 0 degrees
- moved Q1 6.98 mm to (107.3, 110.5)
- moved D1 4.07 mm to (107.3, 123.8)
- moved R1 2.54 mm to (107.3, 114.3), turned to 0 degrees
Connections:
- net VCC renamed +5V
- IC1 pad 2: (no net) -> Net-(IC1-Pad2)
- IC1 pad 3: (no net) -> Net-(IC1-Pad3)
- R1 pad 2: Net-(CON1-Pad1) -> Net-(IC1-Pad2)
Routing:
- net Net-(CON1-Pad1): track 40.1 -> 8.04 mm
- net +5V: track 21.9 -> 40.4 mm
- net Net-(D1-Pad1): track 4.45 -> 9.94 mm
- net Net-(IC1-Pad2): track 0.00 -> 5.13 mm
- net Net-(D1-Pad2): track 9.83 -> 13.3 mm
- net (no net): track 2.54 -> 0.00 mm
- net Net-(Q1-Pad2): track 8.41 -> 7.40 mm
